File: hardware/kicad_docs/stm32l0_mod_source.kicad_pcb (KiCad board)
At the start: 4 copper layers, 27.9 x 20.3 mm, 23 parts, among them J1 inputs, J3 SWD_header, J4 signal_outputs, U1 LD3985M33R_SOT23, U2 STM32L031F4Px, U3 MCP4822

Commit message: refine pcb
Routing:
- net GND: track 23.4 -> 23.9 mm
- added copper zone on VDD_layer, net +3V3
- added copper zone on GND_layer, net GND
- removed copper zone on In1.Cu, net +3V3
- removed copper zone on In2.Cu, net GND
Other:
- board text added: "STM32L0 mod source"
